Commit message: added joint 5 revolute and stub

File: robot_moveit_config/config/spotarm_assembly.ros2_control.xacro (robot description, xacro)
@@ -36,4 +36,11 @@
                 <state_interface name="velocity"/>
             </joint>
+            <joint name="Revolute5">
+                <command_interface name="position"/>
+                <state_interface name="position">
+                  <param name="initial_value">${initial_positions['Revolute5']}</param>
+                </state_interface>
+                <state_interface name="velocity"/>
+            </joint>
         </ros2_control>
     </xacro:macro>

File: spotarm_assembly_description/urdf/spotarm_assembly.urdf (robot description, URDF)
Before this commit: robot spotarm_assembly, 5 links, 4 joints
Links:
- added link stub_link, mass 0.2; collision box size=0.02 0.05 0.02; visual box size=0.02 0.3 0.02
- link base_link: geometry collision mesh filename=file:///home/chungus/msd_robot_arm_2/install/spotarm_assemb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 scale=0.001 0.001 0.001; visual mesh filename=file:///home/chungus/msd_robot_arm_2/install/spotarm_assemb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 scale=0.001 0.001 0.001
- link link_2: geometry collision mesh filename=file:///home/chungus/msd_robot_arm_2/install/spotarm_assemb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 scale=0.001 0.001 0.001; visual mesh filename=file:///home/chungus/msd_robot_arm_2/install/spotarm_assemb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 scale=0.001 0.001 0.001
- link link_3: geometry collision mesh filename=file:///home/chungus/msd_robot_arm_2/install/spotarm_assemb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 scale=0.001 0.001 0.001; visual mesh filename=file:///home/chungus/msd_robot_arm_2/install/spotarm_assemb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 scale=0.001 0.001 0.001
- link link_4: geometry collision mesh filename=file:///home/chungus/msd_robot_arm_2/install/spotarm_assemb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 scale=0.001 0.001 0.001; visual mesh filename=file:///home/chungus/msd_robot_arm_2/install/spotarm_assemb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 scale=0.001 0.001 0.001
- link link_5: geometry collision mesh filename=file:///home/chungus/msd_robot_arm_2/install/spotarm_assemb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 scale=0.001 0.001 0.001; visual mesh filename=file:///home/chungus/msd_robot_arm_2/install/spotarm_assemb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 scale=0.001 0.001 0.001
Joints:
- added joint Revolute5: type continuous, parent link_5, child stub_link, origin xyz=0.07 -0.144 0 rpy=0 0 0, axis 1.0 0.0 0.0

File: spotarm_assembly_description/urdf/spotarm_assembly.xacro (robot description, xacro)
@@ -104,4 +104,24 @@
   </collision>
 </link>
+<link name="stub_link">
+  <inertial>
+    <origin xyz="0.011 0 0" rpy="0 0 0"/>
+    <mass value="0.2"/>
+    <inertia ixx="1.3333333333333334e-05" iyy="4.8333333333333334e-05" izz="4.8333333333333334e-05" ixy="0.0" iyz="0.0" ixz="0.0"/>
+  </inertial>
+  <visual>
+    <origin xyz="0.011 -0.14 0" rpy="0 0 0"/>
+    <geometry>
+      <box size="0.02 0.3 0.02"/>
+    </geometry>
+    <material name="silver"/>
+  </visual>
+  <collision>
+    <origin xyz="0.011 0 0" rpy="0 0 0"/>
+    <geometry>
+      <box size="0.02 0.05 0.02"/>
+    </geometry>
+  </collision>
+</link>
 <joint name="Revolute1" type="continuous">
   <origin xyz="0.02835 -0.011972 0.033179" rpy="0 0 0"/>
@@ -128,3 +148,9 @@
   <axis xyz="-0.0 -1.0 0.0"/>
 </joint>
+<joint name="Revolute5" type="continuous">
+  <origin xyz="0.07 -0.144 0" rpy="0 0 0"/>
+  <parent link="link_5"/>
+  <child link="stub_link"/>
+  <axis xyz="1.0 0.0 0.0"/>
+</joint>
 </robot>
